Commit message: update

File: assets/robot/robot.urdf (robot description, URDF)
Before this commit: robot NexArm-sim, 11 links, 10 joints
Joints:
- joint left_jaw_slide_joint: limit lower=0.0 upper=0.02 effort=1000000 velocity=1000000 -> lower=0.0 upper=0.0255 effort=1000000 velocity=1000000
- joint right_jaw_slide_joint: limit lower=-0.02 upper=0.0 effort=1000000 velocity=1000000 -> lower=-0.0255 upper=0.0 effort=1000000 velocity=1000000
